Commit message: intel d435i tf

File: lgdxrobot2-description/src/description/lgdxrobot2_description.urdf (robot description, URDF)
Before this commit: robot lgdxrobot2, 2 links, 1 joints
Links:
- added link camera_centre_link; collision box size=${camera_length} ${camera_width} ${camera_height}; visual box size=${camera_length} ${camera_width} ${camera_height}
- added link camera_link
Joints:
- added joint camera_centre_joint: type fixed, parent camera_centre_link, child camera_link, origin xyz=${camera_centre_xoff} ${camera_centre_yoff} ${camera_centre_zoff}
- added joint camera_joint: type fixed, parent base_link, child camera_centre_link, origin xyz=${camera_xoff} ${camera_yoff} ${camera_zoff}
