Commit message: change launch file for description

File: lgdxrobot2_webots/resource/lgdxrobot2.urdf (robot description, URDF)
Before this commit: robot LGDXRobot2, 19 links, 18 joints
Links:
- removed link BASE_CENTRE_SOLID
- removed link BASE_FRONT_SOLID
- removed link BASE_REAR_SOLID
- removed link BASE_TOP_SOLID
- removed link WHEEL_1_SOLID
- removed link WHEEL_2_SOLID
- removed link WHEEL_3_SOLID
- removed link WHEEL_4_SOLID
- removed link base_link
- removed link camera
- removed link camera depth
- removed link camera rgb
- removed link lidar
- removed link lower
- removed link screw0
- removed link screw1
- removed link screw2
- removed link screw3
- removed link solid
Joints:
- removed joint base_link_BASE_CENTRE_SOLID_joint
- removed joint base_link_BASE_FRONT_SOLID_joint
- removed joint base_link_BASE_REAR_SOLID_joint
- removed joint base_link_BASE_TOP_SOLID_joint
- removed joint base_link_camera_joint
- removed joint base_link_lidar_joint
- removed joint camera_camera depth_joint
- removed joint camera_camera rgb_joint
- removed joint lidar_main_motor
- removed joint lidar_screw0_joint
- removed joint lidar_screw1_joint
- removed joint lidar_screw2_joint
- removed joint lidar_screw3_joint
- removed joint lidar_secondary_motor
- removed joint wheel1
- removed joint wheel2
- removed joint wheel3
- removed joint wheel4
