Commit message: update robot

File: lgdxrobot2_description/src/description/lgdxrobot2_simulation.urdf (robot description, URDF)
Before this commit: robot LGDXRobot2, 19 links, 18 joints
Links:
- added link base_footprint
Joints:
- added joint base_joint: type fixed, parent base_link, child base_footprint, origin xyz=0.0 0.0 0.0 rpy=0 0 0
- joint base_link_BASE_CENTRE_SOLID_joint: origin xyz=0 0 -0.036 rpy=0 0 0 -> xyz=0 0 0.057 rpy=0 0 0
- joint base_link_BASE_FRONT_SOLID_joint: origin xyz=0.102 0.00001 -0.036 rpy=0 0 0 -> xyz=0.102 0 0.057 rpy=0 0 0
- joint base_link_BASE_REAR_SOLID_joint: origin xyz=-0.102 0 -0.036 rpy=0 0 0 -> xyz=-0.102 0 0.057 rpy=0 0 0
- joint base_link_BASE_TOP_SOLID_joint: origin xyz=0 0 0.036 rpy=0 0 0 -> xyz=0 0 0.129 rpy=0 0 0
- joint base_link_camera_joint: origin xyz=0.1 0.01 -0.03 rpy=0 0 0 -> xyz=0.1 0.01 0.059 rpy=0 0 0
- joint base_link_lidar_joint: origin xyz=0 0 0.067 rpy=0 0 0 -> xyz=0 0 0.157 rpy=0 0 3.14159
- joint wheel1: origin xyz=0.1055 0.10251 -0.0545 rpy=1.5708 0 0 -> xyz=0.1055 0.1025 0.0375 rpy=1.5708 0 0
- joint wheel2: origin xyz=0.1055 -0.10249 -0.0545 rpy=1.5708 0 0 -> xyz=0.1055 -0.1025 0.0375 rpy=1.5708 0 0
- joint wheel3: origin xyz=-0.1055 0.10251 -0.0545 rpy=1.5708 0 0 -> xyz=-0.1055 0.1025 0.0375 rpy=1.5708 0 0
- joint wheel4: origin xyz=-0.1055 -0.1025 -0.0545 rpy=1.5708 0 0 -> xyz=-0.1055 -0.1025 0.0375 rpy=1.5708 0 0

Commit message: move the robot

File: lgdxrobot2_description/src/description/lgdxrobot2_simulation.urdf (robot description, URDF)
Before this commit: robot LGDXRobot2, 20 links, 19 joints
Links:
- removed link lower
- removed link screw0
- removed link screw1
- removed link screw2
- removed link screw3
- removed link solid
Joints:
- removed joint lidar_main_motor
- removed joint lidar_screw0_joint
- removed joint lidar_screw1_joint
- removed joint lidar_screw2_joint
- removed joint lidar_screw3_joint
- removed joint lidar_secondary_motor
- joint wheel1: type continuous -> fixed
- joint wheel2: type continuous -> fixed
- joint wheel3: type continuous -> fixed
- joint wheel4: type continuous -> fixed
