Commit message: add imu link, sim switch

File: lgdxrobot2_description/description/lgdxrobot2_sim.urdf (robot description, URDF)
Before this commit: robot lgdxrobot2, 9 links, 8 joints
Links:
- added link camera_color_frame
- added link camera_depth_frame
Joints:
- added joint camera_color_frame_joint: type fixed, parent camera_link, child camera_color_frame, origin xyz=-0.00000 0.01500 0.00000 rpy=0.00000 0.00000 0.00000
- added joint camera_depth_frame_joint: type fixed, parent camera_link, child camera_depth_frame, origin xyz=-0.00000 -0.00000 0.00000 rpy=0.00000 0.00000 0.00000

Commit message: spawn robot

File: lgdxrobot2_description/description/lgdxrobot2_sim.urdf (robot description, URDF)
Before this commit: robot lgdxrobot2, 11 links, 10 joints
Links:
- link base_link: mass None -> 2.2768
- link wheel1_link: mass None -> 0.1018
- link wheel2_link: mass None -> 0.1018
- link wheel3_link: mass None -> 0.1018
- link wheel4_link: mass None -> 0.1018

Commit message: move robot

File: lgdxrobot2_description/description/lgdxrobot2_sim.urdf (robot description, URDF)
Before this commit: robot lgdxrobot2, 11 links, 10 joints
Links:
- link base_link: geometry collision box size=0.24000 0.24000 0.07800; visual mesh filename=package://lgdxrobot2_description/meshes/dae/b_Coupling_Nut_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 scale=1.00000 1.00000 1.00000
- link wheel1_link: geometry collision sphere radius=0.03750; visual mesh filename=package://lgdxrobot2_description/meshes/dae/b_Wheel_1_001_.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 scale=1.00000 1.00000 1.00000
- link wheel2_link: geometry collision sphere radius=0.03750; visual mesh filename=package://lgdxrobot2_description/meshes/dae/b_Wheel_2_001_.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 scale=1.00000 1.00000 1.00000
- link wheel3_link: geometry collision sphere radius=0.03750; visual mesh filename=package://lgdxrobot2_description/meshes/dae/b_Wheel_3_001_.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 scale=1.00000 1.00000 1.00000
- link wheel4_link: geometry collision sphere radius=0.03750; visual mesh filename=package://lgdxrobot2_description/meshes/dae/b_Wheel_4_001_.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 scale=1.00000 1.00000 1.00000
Joints:
- joint wheel1_link_joint: axis 0.00000 0.00000 1.00000 -> 0 0 1; limit effort=30.00000 velocity=12.00000 -> effort=10000 velocity=10
- joint wheel2_link_joint: axis 0.00000 0.00000 1.00000 -> 0 0 1; limit effort=30.00000 velocity=12.00000 -> effort=10000 velocity=10
- joint wheel3_link_joint: axis 0.00000 0.00000 1.00000 -> 0 0 1; limit effort=30.00000 velocity=12.00000 -> effort=10000 velocity=10
- joint wheel4_link_joint: axis 0.00000 0.00000 1.00000 -> 0 0 1; limit effort=30.00000 velocity=12.00000 -> effort=10000 velocity=10

Commit message: fix gz settings

File: lgdxrobot2_description/description/lgdxrobot2_sim.urdf (robot description, URDF)
Before this commit: robot lgdxrobot2, 11 links, 10 joints
Links:
- link wheel1_link: geometry collision sphere radius=0.0375; visual mesh filename=package://lgdxrobot2_description/meshes/dae/b_Wheel_1_001_.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 scale=1.00000 1.00000 1.00000
- link wheel2_link: geometry collision sphere radius=0.0375; visual mesh filename=package://lgdxrobot2_description/meshes/dae/b_Wheel_2_001_.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 scale=1.00000 1.00000 1.00000
- link wheel3_link: geometry collision sphere radius=0.0375; visual mesh filename=package://lgdxrobot2_description/meshes/dae/b_Wheel_3_001_.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 scale=1.00000 1.00000 1.00000
- link wheel4_link: geometry collision sphere radius=0.0375; visual mesh filename=package://lgdxrobot2_description/meshes/dae/b_Wheel_4_001_.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 scale=1.00000 1.00000 1.00000
Joints:
- joint wheel2_link_joint: origin xyz=0.08185 -0.10362 0.03676 rpy=-1.57080 0.00000 0.00000 -> xyz=0.08185 -0.10362 0.03681 rpy=-1.57080 0.00000 0.00000
