Commit message: fix urdf webots bug

File: lgdxrobot2_description/description/lgdxrobot2.urdf (robot description, URDF)
Before this commit: robot lgdxrobot2, 7 links, 6 joints
Links:
- added link base_footprint
Joints:
- added joint base_footprint_joint: type fixed, parent base_link, child base_footprint, origin xyz=0.00000 0.00000 0.00000 rpy=0.00000 0.00000 0.00000

Commit message: send joint state

File: lgdxrobot2_description/description/lgdxrobot2.urdf (robot description, URDF)
Before this commit: robot lgdxrobot2, 8 links, 7 joints
Joints:
- joint wheel1_link_joint: axis 0.00000 0.00000 -1.00000 -> 0.00000 0.00000 1.00000
- joint wheel2_link_joint: axis 0.00000 0.00000 -1.00000 -> 0.00000 0.00000 1.00000
- joint wheel3_link_joint: axis 0.00000 0.00000 -1.00000 -> 0.00000 0.00000 1.00000
- joint wheel4_link_joint: axis 0.00000 0.00000 -1.00000 -> 0.00000 0.00000 1.00000

Commit message: raise the lidar

File: lgdxrobot2_description/description/lgdxrobot2.urdf (robot description, URDF)
Before this commit: robot lgdxrobot2, 8 links, 7 joints
Joints:
- joint lidar_link_joint: origin xyz=0.06000 -0.00000 0.13331 rpy=0.00000 0.00000 0.00000 -> xyz=0.06000 -0.00000 0.15641 rpy=0.00000 0.00000 0.00000

Commit message: camera position

File: lgdxrobot2_description/description/lgdxrobot2.urdf (robot description, URDF)
Before this commit: robot lgdxrobot2, 8 links, 7 joints
Links:
- added link camera_color_frame_sim
- added link camera_depth_frame_sim
Joints:
- added joint camera_color_frame_joint: type fixed, parent camera_link, child camera_color_frame_sim, origin xyz=-0.00000 0.01500 0.00000 rpy=0.00000 0.00000 0.00000
- added joint camera_depth_frame_joint: type fixed, parent camera_link, child camera_depth_frame_sim, origin xyz=-0.00000 -0.00000 0.00000 rpy=0.00000 0.00000 0.00000
- joint camera_link_joint: origin xyz=0.10800 0.00026 0.05931 rpy=0.00000 0.00000 0.00000 -> xyz=0.13104 0.01776 0.07181 rpy=0.00000 0.00000 0.00000

Commit message: reverse lidar

File: lgdxrobot2_description/description/lgdxrobot2.urdf (robot description, URDF)
Before this commit: robot lgdxrobot2, 10 links, 9 joints
Joints:
- joint lidar_link_joint: origin xyz=0.06000 -0.00000 0.15641 rpy=0.00000 0.00000 0.00000 -> xyz=0.06000 -0.00000 0.15641 rpy=0.00000 0.00000 -3.14159

Commit message: update description

File: lgdxrobot2_description/description/lgdxrobot2.urdf (robot description, URDF)
Before this commit: robot lgdxrobot2, 9 links, 8 joints
Joints:
- joint imu_link_joint: origin xyz=-0.08351 0.00000 0.09830 rpy=0.00000 0.00000 0.00000 -> xyz=-0.08351 0.00000 0.0649 rpy=0.00000 0.00000 0.00000

File: lgdxrobot2_description/description/lgdxrobot2_sim.urdf (robot description, URDF)
Before this commit: robot lgdxrobot2, 11 links, 10 joints
Joints:
- joint imu_link_joint: origin xyz=-0.08351 0.00000 0.09830 rpy=0.00000 0.00000 0.00000 -> xyz=-0.08351 0.00000 0.0649 rpy=0.00000 0.00000 0.00000

Commit message: fiz gz cam

File: lgdxrobot2_description/description/lgdxrobot2.urdf (robot description, URDF)
Before this commit: robot lgdxrobot2, 9 links, 8 joints
Joints:
- joint wheel2_link_joint: origin xyz=0.08185 -0.10362 0.03676 rpy=-1.57080 0.00000 0.00000 -> xyz=0.08200 -0.10357 0.03681 rpy=-1.57080 0.00000 0.00000

File: lgdxrobot2_description/description/lgdxrobot2_sim.urdf (robot description, URDF)
Before this commit: robot lgdxrobot2, 11 links, 10 joints
Joints:
- joint wheel2_link_joint: origin xyz=0.08185 -0.10362 0.03681 rpy=-1.57080 0.00000 0.00000 -> xyz=0.08200 -0.10357 0.03681 rpy=-1.57080 0.00000 0.00000

Commit message: fix udrf

File: lgdxrobot2_description/description/lgdxrobot2.urdf (robot description, URDF)
Before this commit: robot lgdxrobot2, 9 links, 8 joints
Links:
- link base_link: geometry visual mesh filename=package://lgdxrobot2_description/meshes/dae/b_Coupling_Nut_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 scale=1.00000 1.00000 1.00000; visual mesh filename=package://lgdxrobot2_description/meshes/dae/b_LGDXRobot2_Bo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 scale=1.00000 1.00000 1.00000
- link camera_link: geometry visual mesh filename=package://lgdxrobot2_description/meshes/dae/b_Camera_001_.d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 scale=1.00000 1.00000 1.00000
- link lidar_link: geometry visual mesh filename=package://lgdxrobot2_description/meshes/dae/b_Lidar_001_.dae scale=1.00000 1.00000 1.00000
- link wheel1_link: geometry visual mesh filename=package://lgdxrobot2_description/meshes/dae/b_Wheel_1_001_.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 scale=1.00000 1.00000 1.00000
- link wheel2_link: geometry visual mesh filename=package://lgdxrobot2_description/meshes/dae/b_Wheel_2_001_.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 scale=1.00000 1.00000 1.00000
- link wheel3_link: geometry visual mesh filename=package://lgdxrobot2_description/meshes/dae/b_Wheel_3_001_.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 scale=1.00000 1.00000 1.00000
- link wheel4_link: geometry visual mesh filename=package://lgdxrobot2_description/meshes/dae/b_Wheel_4_001_.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 scale=1.00000 1.00000 1.00000

File: lgdxrobot2_description/description/lgdxrobot2_sim.urdf (robot description, URDF)
Before this commit: robot lgdxrobot2, 11 links, 10 joints
Links:
- link camera_link: geometry visual mesh filename=package://lgdxrobot2_description/meshes/dae/b_Camera_001_.d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 scale=1.00000 1.00000 1.00000
- link lidar_link: geometry visual mesh filename=package://lgdxrobot2_description/meshes/dae/b_Lidar_001_.dae scale=1.00000 1.00000 1.00000
